File: 10BASE-T1L_2.sch (EAGLE design)
At the start: 163 parts, among them J1 10104110-0001LF, J2 A-2004-2-4-LPS-N-R, J3 TBL009-254-03GY-2GY, J4 TBL009-254-02GY-2GY, T1 ALT4532M-201-T001, T4 H1102NLT, U1 DP83TD510ERHBR, U2 DP83822IRHBR, U3 CO32H4-25.000-33GDTST, U4 LMR38020SDDAR, U5 SN74LVC1G17DCKR, U6 SN74LVC1G17DCKR

Commit message: adding reset cap
Parts:
- added C61: 10nF, ruark2:0402_CAPACITOR
- R68: value 100k -> 115k
- R69: value 24.9k -> 49.9k
Connections:
- net !RST: now also C61.1
- net GND: now also C61.2
Changed lines of the file:
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@@
 <part name="C56" library="rcl" library_urn="urn:adsk.eagle:library:334" deviceset="C-EU" device="C1206" package3d_urn="urn:adsk.eagle:package:23618/2" value="22uF"/>
 <part name="C57" library="rcl" library_urn="urn:adsk.eagle:library:334" deviceset="C-EU" device="C1206" package3d_urn="urn:adsk.eagle:package:23618/2" value="22uF"/>
-<part name="R68" library="ruark2" deviceset="0603_RESISTOR" device="" value="100k"/>
-<part name="R69" library="ruark2" deviceset="0603_RESISTOR" device="" value="24.9k"/>
+<part name="R68" library="ruark2" deviceset="0603_RESISTOR" device="" value="115k"/>
+<part name="R69" library="ruark2" deviceset="0603_RESISTOR" device="" value="49.9k"/>
 <part name="GND71" library="supply1" library_urn="urn:adsk.eagle:library:371" deviceset="GND" device=""/>
 <part name="GND72" library="supply1" library_urn="urn:adsk.eagle:library:371" deviceset="GND" device=""/>
@@
 <part name="+3V19" library="supply1" library_urn="urn:adsk.eagle:library:371" deviceset="+3V3" device=""/>
 <part name="+3V21" library="supply1" library_urn="urn:adsk.eagle:library:371" deviceset="+3V3" device=""/>
+<part name="C61" library="ruark2" deviceset="0402_CAPACITOR" device="" value="10nF"/>
+<part name="GND86" library="supply1" library_urn="urn:adsk.eagle:library:371" deviceset="GND" device=""/>
 </parts>
 <sheets>
@@
 <attribute name="VALUE" x="236.22" y="17.78" size="1.778" layer="96" rot="R90"/>
 </instance>
+<instance part="C61" gate="G$1" x="127" y="71.12" smashed="yes">
+<attribute name="NAME" x="128.524" y="74.041" size="1.778" layer="95"/>
+<attribute name="VALUE" x="128.524" y="68.961" size="1.778" layer="96"/>
+</instance>
+<instance part="GND86" gate="1" x="127" y="63.5" smashed="yes">
+<attribute name="VALUE" x="124.46" y="60.96" size="1.778" layer="96"/>
+</instance>
 </instances>
 <busses>
@@
 <pinref part="C60" gate="G$1" pin="2"/>
 <pinref part="GND85" gate="1" pin="GND"/>
+</segment>
+<segment>
+<pinref part="GND86" gate="1" pin="GND"/>
+<pinref part="C61" gate="G$1" pin="2"/>
+<wire x1="127" y1="66.04" x2="127" y2="68.58" width="0.1524" layer="91"/>
 </segment>
 </net>
@@
 <wire x1="160.02" y1="93.98" x2="139.7" y2="93.98" width="0.1524" layer="91"/>
 <wire x1="139.7" y1="93.98" x2="139.7" y2="78.74" width="0.1524" layer="91"/>
-<wire x1="139.7" y1="78.74" x2="111.76" y2="78.74" width="0.1524" layer="91"/>
+<wire x1="139.7" y1="78.74" x2="127" y2="78.74" width="0.1524" layer="91"/>
 <label x="111.76" y="78.74" size="1.778" layer="95"/>
-</segment>
-<segment>
+<pinref part="C61" gate="G$1" pin="1"/>
+<wire x1="127" y1="78.74" x2="111.76" y2="78.74" width="0.1524" layer="91"/>
+<wire x1="127" y1="76.2" x2="127" y2="78.74" width="0.1524" layer="91"/>
+<junction x="127" y="78.74"/>
+</segment>
+<segment>

Commit message: Added PD detection
Parts:
- removed R65: 75, ruark2:0603_RESISTOR
- added C62: 0.1uF, ruark2:0402_CAPACITOR
- added D11, D12: (no value), diode:DIODE-MINIMELF
- added D5, D7, D8: SM4007PL, ruark2:SM4007PL
- added D9: CJ431, ruark2:CJ431
- added Q1, Q2, Q3: MMBT5551, ruark2:MMBT3904-TPCENTERED
- added Q4: MMBT5401, ruark2:MMBT3906-7-FCENTERED
- added Q5: AO3400A, ruark2:AO3400A
- added R60, R63: 75, ruark2:0402_RESISTOR
- added R71, R72, R73, R74: 1M, ruark2:0603_RESISTOR
- added R75: 10k, ruark2:0402_RESISTOR
- added R76: 100k, ruark2:0402_RESISTOR
- added R77, R79: 1M, ruark2:0402_RESISTOR
- added R80: 10M, ruark2:0402_RESISTOR
- R32, R33: device ruark2:0603_RESISTOR -> ruark2:0402_RESISTOR
- R64: value 75 -> 0R; device ruark2:0603_RESISTOR -> ruark2:1206_RESISTOR
Connections:
- removed net RX+: J2.3, T4.2P
- removed net RX-: J2.6, T4.2N
- removed net TX+: J2.1, T4.1P
- removed net TX-: J2.2, T4.1N
- new net N$11: Q4.C, R75.2
- new net N$20: D9.REF, R73.1, R74.2
- new net N$21: D7.K, D8.K, F1.P$1
- new net N$28: Q3.B, R75.1, R76.2
- new net N$35: Q1.C, Q4.B, R71.1
- new net N$39: Q1.B, Q2.C, R72.1
- new net N$41: D11.A, R77.2, R79.1, R80.2
- new net N$44: Q2.B, R79.2
- new net N$45: D12.C, Q5.G, R77.1
- new net N$7: C62.2, D9.A, Q3.C, R74.1
- new net N$8: C14.1, D5.K, D8.A, L1.2OUT
- new net RTN: D5.A, D6.A, Q1.E, Q2.E, Q3.E, Q5.D, R76.1, R80.1
- new net RX_N: J2.2, T4.2N
- new net RX_P: J2.1, T4.2P
- new net TX_N: J2.6, T4.1N
- new net TX_P: J2.3, T4.1P
- new net V+R: C17.1, C38.1, C39.1, C40.1, C41.1, C42.1, C43.1, C44.1, C45.1, C46.1, C50.1, C51.1, C52.1, R64.2, R66.2, U4.VIN
- net BS: now also R60.1, R63.1; no longer R64.1, R65.1
- net GND: now also D12.A, Q5.S; no longer C14.1, D6.A, L1.2OUT
- net N$26: now also D7.A; no longer F1.P$1
- net N$29: now also R32.1; no longer R64.2
- net N$4: now also R63.2; no longer R32.1
- net N$5: now also R60.2; no longer R33.1
- net N$64: now also R33.1; no longer R65.2
- net V+: now also C62.1, D11.C, D9.K, Q4.E, R64.1, R71.2, R72.2, R73.2; no longer C17.1, C38.1, C39.1, C40.1, C41.1, C42.1, C43.1, C44.1, C45.1, C46.1, C50.1, C51.1, C52.1, R66.2, U4.VIN
Other:
- moved on the sheet: D6, R32, R33, R64

Commit message: Rev2
Fixed RGMII clock
Fixed LED package
Fixed 3.3V PoL output voltage
Fixed oscillator footprint
Fixed PoDl
Switched to JLC Available connectors
Fixed common mode chokes.
Parts:
- removed D11, D12: (no value), diode:DIODE-MINIMELF
- removed D9: CJ431, ruark2:CJ431
- removed Q1, Q2, Q3: MMBT5551, ruark2:MMBT3904-TPCENTERED
- removed Q4: MMBT5401, ruark2:MMBT3906-7-FCENTERED
- removed Q5: AO3400A, ruark2:AO3400A
- removed R72, R73, R74: 1M, ruark2:0603_RESISTOR
- removed R75: 10k, ruark2:0402_RESISTOR
- removed R76: 100k, ruark2:0402_RESISTOR
- removed R77, R79: 1M, ruark2:0402_RESISTOR
- removed R80: 10M, ruark2:0402_RESISTOR
- added JP2: (no value), pinhead:PINHD-2X3
- added R65: 1M, ruark2:1206_RESISTOR
- C12, C13: value 0.1uF -> 1nF 1kV; device ruark2:0603_CAPACITOR -> rcl:C-EUC1206
- C62: value 0.1uF -> 1nF 1kV; device ruark2:0402_CAPACITOR -> rcl:C-EUC1206
- J3: value TBL009-254-03GY-2GY -> KF141R-2.54-3P; device ruark2:TBL009-254-03GY-2GY -> ruark2:KF141R-2.54-3P
- J4: value TBL009-254-02GY-2GY -> KF141R-2.54-2P; device ruark2:TBL009-254-02GY-2GY -> ruark2:KF141R-2.54-2P
- R22: value 499 -> 470
- R32, R33, R60, R63: value 75 -> 49.9
- R50: value 1.96k -> 2k
- R51: value 6.2k -> 5.1k
- R52: value 1.96k -> 1.5k
- R57: device ruark2:0603_RESISTOR -> ruark2:1206_RESISTOR
- R62: value 750k -> 100k
- R66: value 1.65M -> 220k
- R67: value 64.9k -> 68k
- R68: value 115k -> 22k
- R69: value 49.9k -> 51k
- R71: value 1M -> DNP
Connections:
- removed net N$11: Q4.C, R75.2
- removed net N$20: D9.REF, R73.1, R74.2
- removed net N$21: D7.K, D8.K, F1.P$1
- removed net N$26: C14.2, D6.K, D7.A, L1.1IN
- removed net N$28: Q3.B, R75.1, R76.2
- removed net N$35: Q1.C, Q4.B, R71.1
- removed net N$39: Q1.B, Q2.C, R72.1
- removed net N$41: D11.A, R77.2, R79.1, R80.2
- removed net N$44: Q2.B, R79.2
- removed net N$45: D12.C, Q5.G, R77.1
- removed net N$7: C62.2, D9.A, Q3.C, R74.1
- removed net N$8: C14.1, D5.K, D8.A, L1.2OUT
- new net EARTH: C11.1, C12.2, C13.2, C62.1, J3.3, R65.2, R71.1
- new net IN+: C14.2, D6.K, D7.A, JP2.6, L1.1IN
- new net IN-: C14.1, D5.K, D8.A, JP2.5, L1.2OUT
- new net V+F: F1.P$1, JP2.4
- new net VIN: D7.K, D8.K, JP2.2
- net CGND: now also R71.2
- net GND: now also C62.2, JP2.3, R65.1; no longer C11.1, C12.1, C13.1, D12.A, J3.3, Q5.S
- net N$17: now also R36.2
- net N$18: now also R35.2
- net N$36: no longer R35.2
- net N$42: now also C12.1; no longer C13.2
- net N$48: now also C13.1; no longer C12.2
- net N$49: no longer R36.2
- net RTN: now also JP2.1; no longer Q1.E, Q2.E, Q3.E, Q5.D, R76.1, R80.1
- net V+: no longer C62.1, D11.C, D9.K, Q4.E, R71.2, R72.2, R73.2
Other:
- note added: "3.32V Set Point"
- note added: "388kHz"
- note added: "COL: Default = FX_EN=0 and PHY_AD0=1 RX_D0: MODE2 = AN_1=0, PHY_AD1=0 RX_D1: MODE4 = EEE disabled and PHY_AD2=1 RX_D2: Default = Fast mode drop disabled and PHY_AD3=0 RX_D3: Default = AN_EN=1 and PHY_AD4=0 LED_0: MODE4 = AN_0=1 CRS: MODE1 = LED_SPEED=0 and LED_CFG=0 RX_ER: MODE3 = RGMII_EN=1 and SD_EN=1. VDDIO*2.45 RX_DV: Default = XI_50=1, RMII_EN=0 FX_EN=0, AN_EN=1, AN_1=0, AN_0=1: 10BASE-Te Ha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"
- note removed: "400kHz"
- note removed: "COL: Default = FX_EN=0 and PHY_AD0=1 RX_D0: MODE2 = AN_1=0, PHY_AD1=0 RX_D1: MODE4 = EEE disabled and PHY_AD2=1 RX_D2: Default = Fast mode drop disabled and PHY_AD3=0 RX_D3: Default = AN_EN=1 and PHY_AD4=0 LED_0: MODE4 = AN_0=1 CRS: MODE1 = LED_SPEED=0 and LED_CFG=0 RX_ER: MODE3 = RGMII_EN=1 and SD_EN=1 RX_DV: Default = XI_50=1, RMII_EN=0 FX_EN=0, AN_EN=1, AN_1=0, AN_0=1: 10BASE-Te Half/Full dupl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"
- moved on the sheet: C12, C13, C62, L3, R35, R36, R71

Commit message: Loss calculations
Other:
- note added: "200uH"
- note added: "Footprint compatible with Wurth 74930000 350uH transformer"
- note added: "PHYs indlude 50R source termination resistors on MAC lines."
Changed lines of the file:
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@@
 <text x="187.96" y="238.76" size="1.778" layer="91">0.4App</text>
 <text x="205.74" y="213.36" size="1.778" layer="91">3.32V Set Point</text>
+<text x="231.14" y="165.1" size="1.778" layer="91">PHYs indlude 50R source termination
+resistors on MAC lines.</text>
+<text x="76.2" y="127" size="1.778" layer="91">200uH</text>
+<text x="73.66" y="81.28" size="1.778" layer="91">Footprint compatible with
+Wurth 74930000 350uH
+transformer</text>
 </plain>
 <instances>
