File: 10BASE-T1L_3.sch (EAGLE design)
At the start: 172 parts, among them J1 10104110-0001LF, J2 A-2004-2-4-LPS-N-R, J3 KF141R-2.54-3P, J4 KF141R-2.54-2P, T1 ALT4532M-201-T001, T4 H1102NLT, U1 DP83TD510ERHBR, U2 DP83822IRHBR, U3 CO32H4-25.000-33GDTST, U4 LMR38020SDDAR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

Commit message: Adding V3 with inductor PoDL
Parts:
- removed L1: 1mH, ruark2:SMCM090605-102
- added L2, L5: 1mH, ruark2:SNR5040TYD102M
Connections:
- removed net N$17: C8.1, L1.2IN, L3.1OUT, R36.2
- removed net N$18: C9.2, L1.1OUT, L3.2OUT, R35.2
- new net IN+L: C9.2, L2.2, L3.2OUT, R35.2
- new net IN-L: C8.1, L3.1OUT, L5.2, R36.2
- net IN+: now also L2.1; no longer L1.1IN
- net IN-: now also L5.1; no longer L1.2OUT
Other:
- note added: "10BASE-T1L Rev3"
- note removed: "10BASE-T1L"
- moved on the sheet: C14

Commit message: V3 Updates
Parts:
- R68: value 22k -> 51k
- R69: value 51k -> 22k
Changed lines of the file:
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@@
 <part name="C56" library="rcl" library_urn="urn:adsk.eagle:library:334" deviceset="C-EU" device="C1206" package3d_urn="urn:adsk.eagle:package:23618/2" value="22uF"/>
 <part name="C57" library="rcl" library_urn="urn:adsk.eagle:library:334" deviceset="C-EU" device="C1206" package3d_urn="urn:adsk.eagle:package:23618/2" value="22uF"/>
-<part name="R68" library="ruark2" deviceset="0603_RESISTOR" device="" value="22k"/>
-<part name="R69" library="ruark2" deviceset="0603_RESISTOR" device="" value="51k"/>
+<part name="R68" library="ruark2" deviceset="0603_RESISTOR" device="" value="51k"/>
+<part name="R69" library="ruark2" deviceset="0603_RESISTOR" device="" value="22k"/>
 <part name="GND71" library="supply1" library_urn="urn:adsk.eagle:library:371" deviceset="GND" device=""/>
 <part name="GND72" library="supply1" library_urn="urn:adsk.eagle:library:371" deviceset="GND" device=""/>
